Commit message: Add gimbal mount demo

File: hector_models/hector_sensors_description/urdf/hokuyo_utm30lx.urdf.xacro (robot description, xacro)
@@ -3,4 +3,87 @@
     <xacro:property name="M_PI" value="3.1415926535897931" />
     <xacro:macro name="hokuyo_utm30lx_model" params="name parent *origin">
+<!--
+      <joint name="${name}_joint" type="continuous">
+        <parent link="${parent}" />
+        <child link="junta1" />
+        <axis xyz="0 1 0" />
+        <dynamics damping="0" friction="0" />
+      </joint>
+      <link name="junta1">
+        <visual>
+          <geometry>
+            <sphere radius="0.01" />
+          </geometry>
+          <origin xyz="0 0 0" rpy="0 0 0" />
+        </visual>
+        <inertial>
+          <mass value="0.025" />
+          <inertia ixx="5.8083e-4" ixy="0" ixz="0" iyy="3.0833e-5" iyz="0" izz="5.9083e-4" />
+          <origin xyz="0 0 0" rpy="0 0 0" />
+        </inertial>
+        <collision>
+          <geometry>
+            <sphere radius="0.01" />
+          </geometry>
+          <origin xyz="0 0 0" rpy="0 0 0" />
+        </collision>
+      </link>
+      <joint name="${name}_joint2" type="continuous">
+        <parent link="junta1" />
+        <child link="junta2" />
+        <axis xyz="0 0 1" />
+        <dynamics damping="0" friction="0" />
+      </joint>
+      <link name="junta2">
+        <visual>
+          <geometry>
+            <sphere radius="0.01" />
+          </geometry>
+          <origin xyz="0 0 -0.01" rpy="0 0 0" />
+        </visual>
+        <inertial>
+          <mass value="0.025" />
+          <inertia ixx="5.8083e-4" ixy="0" ixz="0" iyy="3.0833e-5" iyz="0" izz="5.9083e-4" />
+          <origin xyz="0 0 -0.01" rpy="0 0 0" />
+        </inertial>
+        <collision>
+          <geometry>
+            <sphere radius="0.01" />
+          </geometry>
+          <origin xyz="0 0 -0.01" rpy="0 0 0" />
+        </collision>
+      </link>
+      <joint name="${name}_joint3" type="continuous">
+        <parent link="junta1" />
+        <child link="junta3" />
+        <axis xyz="1 0 0" />
+        <dynamics damping="0" friction="0" />
+      </joint>
+      <link name="junta3">
+        <visual>
+          <geometry>
+            <sphere radius="0.01" />
+          </geometry>
+          <origin xyz="0 0 -0.02" rpy="0 0 0" />
+        </visual>
+        <inertial>
+          <mass value="0.025" />
+          <inertia ixx="5.8083e-4" ixy="0" ixz="0" iyy="3.0833e-5" iyz="0" izz="5.9083e-4" />
+          <origin xyz="0 0 -0.02" rpy="0 0 0" />
+        </inertial>
+        <collision>
+          <geometry>
+            <sphere radius="0.01" />
+          </geometry>
+          <origin xyz="0 0 -0.02" rpy="0 0 0" />
+        </collision>
+      </link>
+      <joint name="${name}_jointfixed" type="fixed">
+        <xacro:insert_block name="origin" />
+        <parent link="junta3"/>
+        <child link="${name}_frame"/>
+      </joint>
+-->
+<!---->
       <joint name="${name}_joint" type="fixed">
         <xacro:insert_block name="origin" />
@@ -8,4 +91,5 @@
         <child link="${name}_frame"/>
       </joint>
+<!---->
       <link name="${name}_frame">
         <inertial>
