Commit message: Update from hector_quadrotor

File: hector_models/hector_sensors_description/urdf/camera360.urdf.xacro (robot description, xacro)
@@ -2,5 +2,8 @@
 <robot xmlns:xacro="http://ros.org/wiki/xacro">
   <xacro:property name="M_PI" value="3.1415926535897931" />
-  <xacro:macro name="camera360" params="name right_cam_name left_cam_name parent *origin *calibration dist_between_cameras ros_topic update_rate res_x res_y image_format fov">
+  <xacro:property name="default_collision_radius" value="0.025" />
+  <xacro:property name="visual_radius" value="0.011" />
+  <xacro:property name="cable_collision_length" value="0.05" />
+  <xacro:macro name="camera360" params="name right_cam_name left_cam_name parent collision_radius:=${default_collision_radius} *origin *calibration dist_between_cameras ros_topic update_rate res_x res_y image_format fov">
     <joint name="${name}_center_joint" type="fixed">
       <xacro:insert_block name="origin" />
@@ -8,5 +11,44 @@
       <child link="${name}_center_link"/>
     </joint>
-    <link name="${name}_center_link" />
+    <link name="${name}_center_link">
+      <!-- Sphere body -->
+      <visual>
+        <origin xyz="0 0 0" rpy="0 0 0"/>
+        <geometry>
+          <sphere radius="${visual_radius}"/>
+        </geometry>
+        <material name="Grey">
+          <color rgba="0.5 0.5 0.5 1"/>
+        </material>
+      </visual>
+      <collision>
+        <origin xyz="0 0 0" rpy="0 0 0"/>
+        <geometry>
+          <sphere radius="${collision_radius}"/>
+        </geometry>
+        <material name="Grey">
+          <color rgba="0.5 0.5 0.5 1"/>
+        </material>
+      </collision>
+      <!-- Cable -->
+<!--      <visual>
+        <origin xyz="${visual_radius + cable_collision_length/2} 0 0" rpy="0 0 0"/>
+        <geometry>
+          <box size="${cable_collision_length} 0.03 0.03"/>
+        </geometry>
+        <material name="Grey">
+          <color rgba="0.5 0.5 0.5 1"/>
+        </material>
+      </visual>-->
+      <collision>
+        <origin xyz="${0.011 + cable_collision_length/2} 0 0" rpy="0 0 0"/>
+        <geometry>
+          <box size="${cable_collision_length} 0.03 0.03"/>
+        </geometry>
+        <material name="Grey">
+          <color rgba="0.5 0.5 0.5 1"/>
+        </material>
+      </collision>
+    </link>
     <joint name="${name}_${right_cam_name}_joint" type="fixed">
       <origin xyz="0 ${dist_between_cameras/2} 0" rpy="${M_PI*0.5} 0 ${-M_PI*0.5}"/>

Commit message: - Fix wrong execution ID in feedback message - Update hector_quadrotor

File: hector_models/hector_sensors_description/urdf/camera360.urdf.xacro (robot description, xacro)
@@ -1,7 +1,7 @@
 <?xml version="1.0"?>
-<robot xmlns:xacro="http://ros.org/wiki/xacro">
+<robot xmlns:xacro="http://www.ros.org/wiki/xacro">
   <xacro:property name="M_PI" value="3.1415926535897931" />
   <xacro:property name="default_collision_radius" value="0.025" />
-  <xacro:property name="visual_radius" value="0.011" />
+  <xacro:property name="visual_radius" value="0.02" />
   <xacro:property name="cable_collision_length" value="0.05" />
   <xacro:macro name="camera360" params="name right_cam_name left_cam_name parent collision_radius:=${default_collision_radius} *origin *calibration dist_between_cameras ros_topic update_rate res_x res_y image_format fov">

File: hector_models/hector_sensors_description/urdf/realsense_d435_camera.urdf.xacro (robot description, xacro)
@@ -8,5 +8,5 @@
   <node pkg="tf" type="static_transform_publisher" name="kinect_base_link2" args="0 0 0 -1.57 0 -1.57 /arm_rgbd_cam_depth_frame /arm_rgbd_cam_depth_optical_frame  100" />
 -->
-<robot xmlns:xacro="http://ros.org/wiki/xacro">
+<robot xmlns:xacro="http://www.ros.org/wiki/xacro">
   <xacro:property name="M_PI" value="3.1415926535897931" />
   <xacro:property name="realsense_d435_width" value="0.09"/>
@@ -35,19 +35,10 @@
           <inertia ixx="5.8083e-4" ixy="0" ixz="0" iyy="3.0833e-5" iyz="0" izz="5.9083e-4" />
         </inertial>
-        <visual>
-          <origin xyz="${realsense_d435_case_offset_x} ${realsense_d435_case_offset_y} ${realsense_d435_case_offset_z}" rpy="0 0 0" />
-          <geometry>
-            <box size="${realsense_d435_depth} ${realsense_d435_width} ${realsense_d435_height}" />
-          </geometry>
-          <material name="DarkGrey">
-            <color rgba="0.3 0.3 0.3 1"/>
-          </material>
-        </visual>
-<!--        <visual>
+	<visual>
           <origin xyz="${realsense_d435_front_to_depth} ${realsense_d435_case_offset_y} 0.0" rpy="${M_PI/2} 0 ${M_PI/2}" />
           <geometry>
-            <mesh filename="package://realsense2_camera/meshes/d435.dae" />
+            <mesh filename="package://hector_sensors_description/meshes/intel_realsense_d435/D435.dae" scale="0.001 0.001 0.001" />
           </geometry>
-        </visual>-->
+        </visual>
         <collision>
           <origin xyz="${realsense_d435_case_offset_x} ${realsense_d435_case_offset_y} ${realsense_d435_case_offset_z}" rpy="0 0 0" />
@@ -121,4 +112,5 @@
     <!--
       Use the macro below for adding the realsense model with link geometry
+      The origin is the left infrared (depth) camera, which is also the origin of the depth image
     -->
     <xacro:macro name="realsense_d435_camera" params="name parent *origin">
@@ -126,4 +118,13 @@
         <xacro:insert_block name="origin" />
       </xacro:realsense_d435_camera_model>
+      <xacro:realsense_d435_camera_gazebo_plugin_macro name="${name}" parent="${parent}" image_topic="image_raw" depth_points_topic="depth/points" min_range="0.3" max_range="9.0" update_rate="20"/>
+    </xacro:macro>
+    <!--
+      Insert the realsense with link geometry. Origin is the mounting hole at the back of the camera.
+    -->
+    <xacro:macro name="realsense_d435_camera_with_mount" params="name parent *origin">
+      <xacro:realsense_d435_camera_model_with_mount name="${name}" parent="${parent}">
+        <xacro:insert_block name="origin" />
+      </xacro:realsense_d435_camera_model_with_mount>
       <xacro:realsense_d435_camera_gazebo_plugin_macro name="${name}" parent="${parent}" image_topic="image_raw" depth_points_topic="depth/points" min_range="0.3" max_range="9.0" update_rate="20"/>
     </xacro:macro>

File: hector_models/hector_sensors_description/urdf/seek_thermal_compact.urdf.xacro (robot description, xacro)
@@ -1,6 +1,6 @@
 <?xml version="1.0" encoding="UTF-8"?>
-<robot xmlns:xacro="http://ros.org/wiki/xacro">
+<robot xmlns:xacro="http://www.ros.org/wiki/xacro">
   <xacro:include filename="$(find hector_xacro_tools)/urdf/sensor_macros.urdf.xacro" />
-  <xacro:macro name="seek_thermal_compact_camera_model" params="name parent *origin">
+  <xacro:macro name="seek_thermal_compact_camera_model" params="name parent *origin add_geometry">
     <joint name="${name}_joint" type="fixed">
       <xacro:insert_block name="origin" />
@@ -10,40 +10,42 @@
     <link name="${name}_frame">
       <xacro:inertial_sphere mass="0.03" diameter="0.02" />
-      <visual>
-        <origin xyz="0 0.0 -0.025" rpy="0 0 0" />
-        <geometry>
-          <box size="0.02 0.03 0.0375" />
-        </geometry>
-        <material name="DarkGrey">
-          <color rgba="0.3 0.3 0.3 1" />
-        </material>
-      </visual>
-      <visual>
-        <origin xyz="0 0 0" rpy="0 ${M_PI/2} 0" />
-        <geometry>
-          <cylinder length="0.02" radius="0.017" />
-        </geometry>
-        <material name="DarkGrey" />
-      </visual>
-      <visual>
-        <origin xyz="0.01 0 0" rpy="0 ${M_PI/2} 0" />
-        <geometry>
-          <cylinder length="0.018" radius="0.011" />
-        </geometry>
-        <material name="DarkGrey" />
-      </visual>
-      <collision>
-        <origin xyz="0.0055 0 -0.013375" rpy="0 0 0" />
-        <geometry>
-          <box size="0.031 0.034 0.06075" />
-        </geometry>
-      </collision>
-      <xacro:if value="$(arg add_raycast_self_filter_geom)">
+      <xacro:if value="${add_geometry}">
+        <visual>
+            <origin xyz="0 0.0 -0.025" rpy="0 0 0" />
+            <geometry>
+            <box size="0.02 0.03 0.0375" />
+            </geometry>
+            <material name="DarkGrey">
+            <color rgba="0.3 0.3 0.3 1" />
+            </material>
+        </visual>
+        <visual>
+            <origin xyz="0 0 0" rpy="0 ${M_PI/2} 0" />
+            <geometry>
+            <cylinder length="0.02" radius="0.017" />
+            </geometry>
+            <material name="DarkGrey" />
+        </visual>
+        <visual>
+            <origin xyz="0.01 0 0" rpy="0 ${M_PI/2} 0" />
+            <geometry>
+            <cylinder length="0.018" radius="0.011" />
+            </geometry>
+            <material name="DarkGrey" />
+        </visual>
         <collision>
-          <origin xyz="0.0055 0 -0.013375" rpy="0 0 0" />
-          <geometry>
-            <cylinder length="0.06075" radius="0.023"/>
-          </geometry>
+            <origin xyz="0.0055 0 -0.013375" rpy="0 0 0" />
+            <geometry>
+            <box size="0.031 0.034 0.06075" />
+            </geometry>
         </collision>
+        <xacro:if value="$(arg add_raycast_self_filter_geom)">
+            <collision>
+            <origin xyz="0.0055 0 -0.013375" rpy="0 0 0" />
+            <geometry>
+                <cylinder length="0.06075" radius="0.023"/>
+            </geometry>
+            </collision>
+        </xacro:if>
       </xacro:if>
     </link>
@@ -53,8 +55,5 @@
     </gazebo>
   </xacro:macro>
-  <xacro:macro name="seek_thermal_compact_camera" params="name parent *origin">
-    <xacro:seek_thermal_compact_camera_model name="${name}" parent="${parent}">
-      <xacro:insert_block name="origin" />
-    </xacro:seek_thermal_compact_camera_model>
+  <xacro:macro name="seek_thermal_compact_gazebo_plugin_macro" params="name parent *origin">
     <gazebo reference="${name}_frame">
       <sensor type="camera" name="thermal_camera_sensor">
@@ -83,3 +82,25 @@
     </gazebo>
   </xacro:macro>
+  <xacro:macro name="seek_thermal_compact_camera" params="name parent *origin">
+    <xacro:seek_thermal_compact_camera_model name="${name}" parent="${parent}" add_geometry="true">
+      <xacro:insert_block name="origin" />
+    </xacro:seek_thermal_compact_camera_model>
+    <xacro:seek_thermal_compact_gazebo_plugin_macro name="${name}" parent="${parent}">
+      <xacro:insert_block name="origin" />
+    </xacro:seek_thermal_compact_gazebo_plugin_macro>
+  </xacro:macro>
+  <xacro:macro name="seek_thermal_compact_camera_no_geom" params="name parent *origin">
+    <xacro:seek_thermal_compact_camera_model name="${name}" parent="${parent}" add_geometry="false">
+      <xacro:insert_block name="origin" />
+    </xacro:seek_thermal_compact_camera_model>
+    <xacro:seek_thermal_compact_gazebo_plugin_macro name="${name}" parent="${parent}">
+      <xacro:insert_block name="origin" />
+    </xacro:seek_thermal_compact_gazebo_plugin_macro>
+  </xacro:macro>
+  <xacro:macro name="realsense_camera_no_geom" params="name parent *origin">
+    <xacro:realsense_d435_camera_model_no_geom name="${name}" parent="${parent}">
+      <xacro:insert_block name="origin" />
+    </xacro:realsense_d435_camera_model_no_geom>
+    <xacro:seek_thermal_compact_gazebo_plugin_macro name="${name}" parent="${parent}" image_topic="image_raw" depth_points_topic="depth/points" min_range="0.3" max_range="9.0" update_rate="20"/>
+    </xacro:macro>
 </robot>

File: hector_models/hector_sensors_description/urdf/vlp16.urdf.xacro (robot description, xacro)
@@ -1,4 +1,4 @@
 <?xml version="1.0"?>
-<robot xmlns:xacro="http://ros.org/wiki/xacro">
+<robot xmlns:xacro="http://www.ros.org/wiki/xacro">
     <xacro:property name="M_PI" value="3.1415926535897931" />
     <xacro:macro name="vlp16_model" params="name parent *origin">
@@ -9,9 +9,22 @@
       </joint>
       <link name="${name}_frame">
-        <xacro:inertial_sphere mass="0.8" diameter="0.1033" />
-        <visual>        -->
-          <origin rpy="0 0 0" xyz="0 0 0.0018500"/>
+        <xacro:inertial_sphere mass="0.83" diameter="0.1033" />
+        <!-- Visual geometry by velodyne_simulator https://bitbucket.org/DataspeedInc/velodyne_simulator -->
+        <visual>
+          <origin xyz="0 0 -0.0377" />
           <geometry>
-            <cylinder radius="0.0516" length="0.0717"/>
+            <mesh filename="package://hector_sensors_description/meshes/vlp16/VLP16_base_1.dae" />
+          </geometry>
+        </visual>
+        <visual>
+          <origin xyz="0 0 -0.0377" />
+          <geometry>
+            <mesh filename="package://hector_sensors_description/meshes/vlp16/VLP16_base_2.dae" />
+          </geometry>
+        </visual>
+        <visual>
+          <origin xyz="0 0 -0.0377" />
+          <geometry>
+            <mesh filename="package://hector_sensors_description/meshes/vlp16/VLP16_scan.dae" />
           </geometry>
         </visual>

File: hector_quadrotor/hector_quadrotor_gazebo/urdf/quadrotor_sensors.gazebo.xacro (robot description, xacro)
@@ -1,7 +1,4 @@
 <?xml version="1.0"?>
 <robot xmlns:xacro="http://www.ros.org/wiki/xacro">
-  <!-- Arguments for GPS Sim -->
-  <xacro:arg name="reference_latitude" default="49.860246" />
-  <xacro:arg name="reference_longitude" default="8.687077" />
   <!-- Quadrotor Sensor Plugins -->
   <xacro:macro name="quadrotor_sensors">
@@ -44,6 +41,6 @@
             <topicName>fix</topicName>
             <velocityTopicName>fix_velocity</velocityTopicName>
-            <referenceLatitude>$(arg reference_latitude)</referenceLatitude>
-            <referenceLongitude>$(arg reference_longitude)</referenceLongitude>
+            <referenceLatitude>49.860246</referenceLatitude>
+            <referenceLongitude>8.687077</referenceLongitude>
             <drift>5.0 5.0 5.0</drift>
             <gaussianNoise>0.01 0.01 0.01</gaussianNoise>
