Commit message: Fixed error when launching a quadrotor with Kinect

File: hector_models/hector_components_description/urdf/vision_box_common.urdf.xacro (robot description, xacro)
@@ -42,5 +42,5 @@
     </joint>
     <link name="laser1RollServo">
-      <xacro:inertial_sphere mass="0.1" diameter="0.07"/>
+      <xacro:macro name="inertial_sphere" mass="0.1" diameter="0.07"/>
       <visual>
         <origin xyz="${laser1RollServo_size_x/2} 0.0 0.0" rpy="0 0 0"/>
@@ -65,5 +65,5 @@
     </joint>
     <link name="laser1_link">
-      <xacro:inertial_sphere mass="0.1" diameter="0.07"/>
+      <xacro:macro name="inertial_sphere" mass="0.1" diameter="0.07"/>
       <visual>
         <origin xyz="0.0 0.0 ${laser1_size_z/2}" rpy="0 0 0"/>
@@ -90,5 +90,5 @@
     </joint>
     <link name="cameraYawServo">
-      <xacro:inertial_sphere mass="0.1" diameter="0.07"/>
+      <xacro:macro name="inertial_sphere" mass="0.1" diameter="0.07"/>
       <visual>
         <origin xyz="0.0 0.0 ${cameraYawServo_size_z/2}" rpy="0 0 0"/>
@@ -113,5 +113,5 @@
     </joint>
     <link name="mounting_link">
-      <xacro:inertial_sphere mass="0.05" diameter="0.07"/>
+      <xacro:macro name="inertial_sphere" mass="0.05" diameter="0.07"/>
     </link>
     <xacro:thermaleye_camera_model name="infrared" parent="mounting_link">

File: hector_models/hector_sensors_description/urdf/flir_a35_camera.urdf.xacro (robot description, xacro)
@@ -9,5 +9,5 @@
     </joint>
     <link name="${name}_frame">
-      <xacro:inertial_sphere mass="0.01" diameter="0.07" />
+      <xacro:macro name="inertial_sphere" mass="0.01" diameter="0.07" />
       <visual>
         <origin xyz="${0.106*-0.5} 0 0" rpy="0 0 0" />

File: hector_models/hector_sensors_description/urdf/generic_thermal_camera.urdf.xacro (robot description, xacro)
@@ -9,5 +9,5 @@
     </joint>
     <link name="${name}_frame">
-      <!--        <xacro:inertial_sphere mass="0.01" diameter="0.07" />
+      <!--        <xacro:macro name="inertial_sphere" mass="0.01" diameter="0.07" />
       <visual>
       <origin xyz="0 0 0" rpy="0 0 0" />

File: hector_models/hector_sensors_description/urdf/kinect_camera.urdf.xacro (robot description, xacro)
@@ -9,5 +9,5 @@
       </joint>
       <link name="${name}_link">
-        <xacro:inertial_sphere mass="0.01" diameter="0.07" />
+        <xacro:macro name="inertial_sphere" mass="0.01" diameter="0.07" />
         <visual>
           <origin xyz="0 0 0" rpy="0 0 0" />

File: hector_models/hector_sensors_description/urdf/thermaleye_camera.urdf.xacro (robot description, xacro)
@@ -9,5 +9,5 @@
     </joint>
     <link name="${name}_frame">
-      <xacro:inertial_sphere mass="0.01" diameter="0.07" />
+      <xacro:macro name="inertial_sphere" mass="0.01" diameter="0.07" />
       <visual>
         <origin xyz="0 0 0" rpy="0 0 0" />

Commit message: Update from Hector Quadrotor

File: hector_models/hector_components_description/urdf/vision_box_common.urdf.xacro (robot description, xacro)
@@ -42,5 +42,5 @@
     </joint>
     <link name="laser1RollServo">
-      <xacro:macro name="inertial_sphere" mass="0.1" diameter="0.07"/>
+      <xacro:inertial_sphere mass="0.1" diameter="0.07"/>
       <visual>
         <origin xyz="${laser1RollServo_size_x/2} 0.0 0.0" rpy="0 0 0"/>
@@ -65,5 +65,5 @@
     </joint>
     <link name="laser1_link">
-      <xacro:macro name="inertial_sphere" mass="0.1" diameter="0.07"/>
+      <xacro:inertial_sphere mass="0.1" diameter="0.07"/>
       <visual>
         <origin xyz="0.0 0.0 ${laser1_size_z/2}" rpy="0 0 0"/>
@@ -90,5 +90,5 @@
     </joint>
     <link name="cameraYawServo">
-      <xacro:macro name="inertial_sphere" mass="0.1" diameter="0.07"/>
+      <xacro:inertial_sphere mass="0.1" diameter="0.07"/>
       <visual>
         <origin xyz="0.0 0.0 ${cameraYawServo_size_z/2}" rpy="0 0 0"/>
@@ -113,5 +113,5 @@
     </joint>
     <link name="mounting_link">
-      <xacro:macro name="inertial_sphere" mass="0.05" diameter="0.07"/>
+      <xacro:inertial_sphere mass="0.05" diameter="0.07"/>
     </link>
     <xacro:thermaleye_camera_model name="infrared" parent="mounting_link">

File: hector_models/hector_sensors_description/urdf/flir_a35_camera.urdf.xacro (robot description, xacro)
@@ -1,4 +1,4 @@
 <?xml version="1.0"?>
-<robot xmlns:xacro="http://www.ros.org/wiki/xacro">
+<robot xmlns:xacro="http://ros.org/wiki/xacro">
   <xacro:include filename="$(find hector_xacro_tools)/urdf/sensor_macros.urdf.xacro" />
   <xacro:macro name="flir_a35_camera_model" params="name parent *origin">
@@ -9,5 +9,5 @@
     </joint>
     <link name="${name}_frame">
-      <xacro:macro name="inertial_sphere" mass="0.01" diameter="0.07" />
+      <xacro:inertial_sphere mass="0.01" diameter="0.07" />
       <visual>
         <origin xyz="${0.106*-0.5} 0 0" rpy="0 0 0" />

File: hector_models/hector_sensors_description/urdf/generic_thermal_camera.urdf.xacro (robot description, xacro)
@@ -1,4 +1,4 @@
 <?xml version="1.0"?>
-<robot xmlns:xacro="http://www.ros.org/wiki/xacro">
+<robot xmlns:xacro="http://ros.org/wiki/xacro">
   <xacro:include filename="$(find hector_xacro_tools)/urdf/sensor_macros.urdf.xacro" />
   <xacro:macro name="generic_thermal_camera" params="name parent *origin">
@@ -9,5 +9,5 @@
     </joint>
     <link name="${name}_frame">
-      <!--        <xacro:macro name="inertial_sphere" mass="0.01" diameter="0.07" />
+      <!--        <xacro:inertial_sphere mass="0.01" diameter="0.07" />
       <visual>
       <origin xyz="0 0 0" rpy="0 0 0" />

File: hector_models/hector_sensors_description/urdf/hokuyo_utm30lx.urdf.xacro (robot description, xacro)
@@ -1,89 +1,6 @@
 <?xml version="1.0"?>
-<robot xmlns:xacro="http://www.ros.org/wiki/xacro">
+<robot xmlns:xacro="http://ros.org/wiki/xacro">
     <xacro:property name="M_PI" value="3.1415926535897931" />
     <xacro:macro name="hokuyo_utm30lx_model" params="name parent *origin">
-<!--
-      <joint name="${name}_joint" type="continuous">
-        <parent link="${parent}" />
-        <child link="junta1" />
-        <axis xyz="0 1 0" />
-        <dynamics damping="0" friction="0" />
-      </joint>
-      <link name="junta1">
-        <visual>
-          <geometry>
-            <sphere radius="0.01" />
-          </geometry>
-          <origin xyz="0 0 0" rpy="0 0 0" />
-        </visual>
-        <inertial>
-          <mass value="0.025" />
-          <inertia ixx="5.8083e-4" ixy="0" ixz="0" iyy="3.0833e-5" iyz="0" izz="5.9083e-4" />
-          <origin xyz="0 0 0" rpy="0 0 0" />
-        </inertial>
-        <collision>
-          <geometry>
-            <sphere radius="0.01" />
-          </geometry>
-          <origin xyz="0 0 0" rpy="0 0 0" />
-        </collision>
-      </link>
-      <joint name="${name}_joint2" type="continuous">
-        <parent link="junta1" />
-        <child link="junta2" />
-        <axis xyz="0 0 1" />
-        <dynamics damping="0" friction="0" />
-      </joint>
-      <link name="junta2">
-        <visual>
-          <geometry>
-            <sphere radius="0.01" />
-          </geometry>
-          <origin xyz="0 0 -0.01" rpy="0 0 0" />
-        </visual>
-        <inertial>
-          <mass value="0.025" />
-          <inertia ixx="5.8083e-4" ixy="0" ixz="0" iyy="3.0833e-5" iyz="0" izz="5.9083e-4" />
-          <origin xyz="0 0 -0.01" rpy="0 0 0" />
-        </inertial>
-        <collision>
-          <geometry>
-            <sphere radius="0.01" />
-          </geometry>
-          <origin xyz="0 0 -0.01" rpy="0 0 0" />
-        </collision>
-      </link>
-      <joint name="${name}_joint3" type="continuous">
-        <parent link="junta1" />
-        <child link="junta3" />
-        <axis xyz="1 0 0" />
-        <dynamics damping="0" friction="0" />
-      </joint>
-      <link name="junta3">
-        <visual>
-          <geometry>
-            <sphere radius="0.01" />
-          </geometry>
-          <origin xyz="0 0 -0.02" rpy="0 0 0" />
-        </visual>
-        <inertial>
-          <mass value="0.025" />
-          <inertia ixx="5.8083e-4" ixy="0" ixz="0" iyy="3.0833e-5" iyz="0" izz="5.9083e-4" />
-          <origin xyz="0 0 -0.02" rpy="0 0 0" />
-        </inertial>
-        <collision>
-          <geometry>
-            <sphere radius="0.01" />
-          </geometry>
-          <origin xyz="0 0 -0.02" rpy="0 0 0" />
-        </collision>
-      </link>
-      <joint name="${name}_jointfixed" type="fixed">
-        <xacro:insert_block name="origin" />
-        <parent link="junta3"/>
-        <child link="${name}_frame"/>
-      </joint>
--->
-<!---->
       <joint name="${name}_joint" type="fixed">
         <xacro:insert_block name="origin" />
@@ -91,5 +8,4 @@
         <child link="${name}_frame"/>
       </joint>
-<!---->
       <link name="${name}_frame">
         <inertial>

File: hector_models/hector_sensors_description/urdf/kinect_camera.urdf.xacro (robot description, xacro)
@@ -1,4 +1,4 @@
 <?xml version="1.0"?>
-<robot xmlns:xacro="http://www.ros.org/wiki/xacro">
+<robot xmlns:xacro="http://ros.org/wiki/xacro">
     <xacro:property name="M_PI" value="3.1415926535897931" />
     <xacro:macro name="kinect_camera_model" params="name parent *origin">
@@ -9,5 +9,5 @@
       </joint>
       <link name="${name}_link">
-        <xacro:macro name="inertial_sphere" mass="0.01" diameter="0.07" />
+        <xacro:inertial_sphere mass="0.01" diameter="0.07" />
         <visual>
           <origin xyz="0 0 0" rpy="0 0 0" />

File: hector_models/hector_sensors_description/urdf/thermaleye_camera.urdf.xacro (robot description, xacro)
@@ -1,4 +1,4 @@
 <?xml version="1.0"?>
-<robot xmlns:xacro="http://www.ros.org/wiki/xacro">
+<robot xmlns:xacro="http://ros.org/wiki/xacro">
   <xacro:include filename="$(find hector_xacro_tools)/urdf/sensor_macros.urdf.xacro" />
   <xacro:macro name="thermaleye_camera_model" params="name parent *origin">
@@ -9,5 +9,5 @@
     </joint>
     <link name="${name}_frame">
-      <xacro:macro name="inertial_sphere" mass="0.01" diameter="0.07" />
+      <xacro:inertial_sphere mass="0.01" diameter="0.07" />
       <visual>
         <origin xyz="0 0 0" rpy="0 0 0" />
