Commit message: Update from hector_quadrotor

File: hector_models/hector_components_description/urdf/headlight.urdf.xacro (robot description, xacro)
@@ -25,4 +25,12 @@
             <direction>0 0 -1</direction>
           </light>
+          <inertial>
+            <mass>0.00001</mass>
+            <inertia>
+              <ixx>0.00000001</ixx>
+              <iyy>0.00000001</iyy>
+              <izz>0.00000001</izz>
+            </inertia>
+          </inertial>
           <visual name="light_source_visual">
             <geometry>
