Commit message: Update from hector_quadrotor

File: hector_models/hector_components_description/urdf/autonomy_box.urdf.xacro (robot description, xacro)
@@ -5,4 +5,5 @@
   <xacro:include filename="$(find hector_components_description)/urdf/vlp16_mount.urdf.xacro.xml"/>
   <xacro:include filename="$(find hector_sensors_description)/urdf/camera360.urdf.xacro"/>
+  <xacro:include filename="$(find hector_chilitag_description)/urdf/chilitag.urdf.xacro"/>
 <!--  <xacro:arg name="add_self_filter_geom" default="0"/>-->
   <!--<xacro:property name="add_self_filter_geom" value="${arg add_self_filter_geom}"/>-->
@@ -22,8 +23,8 @@
   <xacro:property name="chilitag_white_border" value="0.005"/>
   <xacro:property name="chilitag_thickness" value="0.003"/>
-  <xacro:property name="chilitag_28_x" value="${-computer_box_width/2 + 0.01 + chilitag_size/2}"/> <!-- border is bigger on this side -->
-  <xacro:property name="chilitag_28_y" value="${computer_box_width/2 - chilitag_white_border - chilitag_size/2}"/>
-  <xacro:property name="chilitag_28_z" value="${top_protection_bottom + alu_profile_side_length + chilitag_thickness}"/>
-  <xacro:macro name="autonomy_box_macro" params="parent *origin alu_profile_collision_size_factor name:='autonomy_box'">
+  <xacro:property name="chilitag_29_x" value="${-computer_box_width/2 + chilitag_white_border + chilitag_size/2}"/> <!-- border is bigger on this side -->
+  <xacro:property name="chilitag_29_y" value="${-computer_box_width/2 + 2*chilitag_white_border + chilitag_size/2}"/>
+  <xacro:property name="chilitag_29_z" value="${top_protection_bottom + alu_profile_side_length + chilitag_thickness}"/>
+  <xacro:macro name="autonomy_box_macro" params="parent *origin alu_profile_collision_size_factor name:='autonomy_box' imu_link='imu_link'">
     <xacro:arg name="add_containment_self_filter_geom" default="false"/>
     <joint name="${name}_joint" type="fixed">
@@ -130,7 +131,7 @@
       </visual>
       <!-- Chilitags visual -->
-      <xacro:chilitag_visual_sized name="chilitag28" size="${chilitag_size}">
+      <xacro:chilitag_visual_sized name="chilitag29" size="${chilitag_size}">
 <!--        <origin xyz="${chilitag_28_x} ${chilitag_28_y} ${chilitag_28_z}" rpy="0 ${-M_PI/2} 0"/>-->
-        <origin xyz="${chilitag_28_x} ${chilitag_28_y} ${chilitag_28_z}" rpy="${M_PI} ${0} ${M_PI/2}"/>
+        <origin xyz="${chilitag_29_x} ${chilitag_29_y} ${chilitag_29_z}" rpy="${M_PI} ${0} ${-M_PI/2}"/>
       </xacro:chilitag_visual_sized>
       <!-- Computer box-->
@@ -260,7 +261,7 @@
       </xacro:if>
     </link>
-        <!-- Chilitags -->
-    <xacro:chilitag_no_geom name="chilitag28" size="${chilitag_size}" parent="${name}_link">
-        <origin xyz="${chilitag_28_x} ${chilitag_28_y} ${chilitag_28_z}" rpy="${M_PI} ${0} ${M_PI/2}"/>
+    <!-- Chilitags -->
+    <xacro:chilitag_no_geom name="chilitag29" size="${chilitag_size}" parent="${name}_link">
+      <origin xyz="${chilitag_29_x} ${chilitag_29_y} ${chilitag_29_z}" rpy="${M_PI} ${0} ${-M_PI/2}"/>
     </xacro:chilitag_no_geom>
     <!-- IMU -->
@@ -268,19 +269,28 @@
       <origin xyz="0 0 0" rpy="0 0 0"/>
       <parent link="${name}_link" />
-      <child link="imu_link"/>
+      <child link="${imu_link}"/>
     </joint>
-    <link name="imu_link">
+    <link name="${imu_link}">
     </link>
     <!-- Spinning VLP16 -->
     <xacro:spinning_sensor_mount_macro parent="${name}_link"  name="spin_lidar" scaling="0.001">
-      <origin xyz="0 0 ${0.27 + 0.0944673}" rpy="0.0 0.0 0.0"/>
+      <origin xyz="0 0 ${0.27 + 0.0944673}" rpy="0.0 0.0 ${M_PI}"/>
     </xacro:spinning_sensor_mount_macro>
     <!-- 360 camera -->
     <xacro:camera360 name="camera360" right_cam_name="right" left_cam_name="left" parent="${name}_link" collision_radius="${insta360_collision_radius}" dist_between_cameras="-0.03850784" ros_topic="image_raw" update_rate="10" res_x="1504" res_y="1504" image_format="R8G8B8" fov="${M_PI}">
       <origin xyz="0 0 ${insta360_mounting_height}" rpy="0.0 0 0"/> <!-- base_link to camera mount transform -->
-      <origin xyz="0.00009742  0.00061696 -0.03850784" rpy="3.1373499 -0.0021358 -3.1279404"/> <!-- cam to cam transform (calibration by kalibr) -->
+      <!-- cam to cam transform (calibration by kalibr) -->
+      <!--<origin xyz="0.00009742  0.00061696 -0.03850784" rpy="3.1373499 -0.0021358 -3.1279404"/>--> <!-- insta #1 -->
+      <origin xyz="0.002862424041614364  -0.00013127655875068252 -0.03724378451297336" rpy="-3.1402707 0.0036289 -3.1175768"/> <!-- insta #3 -->
     </xacro:camera360>
-    <gazebo reference="structure_addons_link">
-      <material>Gazebo/Grey</material>
+    <gazebo reference="${name}_link">
+      <visual>
+      <material>
+        <ambient>0.1 0.1 0.1 1</ambient>
+        <diffuse>0.48 0.48 0.48 1</diffuse>
+        <emissive>0.237 0.237 0.237 1</emissive>
+        <specular>0.8 0.8 0.8 1</specular>
+      </material>
+    </visual>
     </gazebo>
   </xacro:macro>

Commit message: Update from hector_quadrotor

File: hector_models/hector_components_description/urdf/autonomy_box.urdf.xacro (robot description, xacro)
@@ -5,8 +5,6 @@
   <xacro:include filename="$(find hector_components_description)/urdf/vlp16_mount.urdf.xacro.xml"/>
   <xacro:include filename="$(find hector_sensors_description)/urdf/camera360.urdf.xacro"/>
-  <xacro:include filename="$(find hector_chilitag_description)/urdf/chilitag.urdf.xacro"/>
 <!--  <xacro:arg name="add_self_filter_geom" default="0"/>-->
   <!--<xacro:property name="add_self_filter_geom" value="${arg add_self_filter_geom}"/>-->
-  <xacro:property name="M_PI" value="3.14159265359"/>
   <xacro:property name="alu_profile_side_length" value="0.02"/>
   <xacro:property name="computer_box_height" value="0.121"/>
@@ -14,17 +12,17 @@
   <xacro:property name="computer_box_length" value="0.19"/>
   <xacro:property name="top_protection_bottom" value="0.4425"/>
-  <xacro:property name="handle_width" value="0.07"/>
-  <xacro:property name="handle_length" value="0.135"/>
-  <xacro:property name="handle_height" value="0.016"/>
-  <xacro:property name="handle_y" value="0.138"/>
   <xacro:property name="insta360_mounting_height" value="0.58"/>
   <xacro:property name="insta360_radius" value="0.011"/>
   <xacro:property name="insta360_collision_radius" value="0.04"/>
-  <xacro:property name="chilitag_white_border" value="0.005"/>
-  <xacro:property name="chilitag_thickness" value="0.003"/>
-  <xacro:property name="chilitag_29_x" value="${-computer_box_width/2 + chilitag_white_border + chilitag_size/2}"/> <!-- border is bigger on this side -->
-  <xacro:property name="chilitag_29_y" value="${-computer_box_width/2 + 2*chilitag_white_border + chilitag_size/2}"/>
-  <xacro:property name="chilitag_29_z" value="${top_protection_bottom + alu_profile_side_length + chilitag_thickness}"/>
-  <xacro:macro name="autonomy_box_macro" params="parent *origin alu_profile_collision_size_factor name:='autonomy_box' imu_link='imu_link'">
+  <xacro:property name="M_PI" value="3.14159265359"/>
+  <xacro:macro name="autonomy_box_macro" params="parent *origin alu_profile_collision_size_factor name:='autonomy_box' imu_link='imu_link' add_chilitags:='true'">
+    <xacro:if value="${add_chilitags}">
+      <xacro:include filename="$(find hector_chilitag_description)/urdf/chilitag.urdf.xacro"/>
+      <xacro:property name="chilitag_white_border" value="0.005"/>
+      <xacro:property name="chilitag_thickness" value="0.003"/>
+      <xacro:property name="chilitag_29_x" value="${-computer_box_width/2 + chilitag_white_border + chilitag_size/2}"/> <!-- border is bigger on this side -->
+      <xacro:property name="chilitag_29_y" value="${-computer_box_width/2 + 2*chilitag_white_border + chilitag_size/2}"/>
+      <xacro:property name="chilitag_29_z" value="${top_protection_bottom + alu_profile_side_length + chilitag_thickness}"/>
+    </xacro:if>
     <xacro:arg name="add_containment_self_filter_geom" default="false"/>
     <joint name="${name}_joint" type="fixed">
@@ -131,8 +129,10 @@
       </visual>
       <!-- Chilitags visual -->
-      <xacro:chilitag_visual_sized name="chilitag29" size="${chilitag_size}">
-<!--        <origin xyz="${chilitag_28_x} ${chilitag_28_y} ${chilitag_28_z}" rpy="0 ${-M_PI/2} 0"/>-->
-        <origin xyz="${chilitag_29_x} ${chilitag_29_y} ${chilitag_29_z}" rpy="${M_PI} ${0} ${-M_PI/2}"/>
-      </xacro:chilitag_visual_sized>
+      <xacro:if value="${add_chilitags}">
+        <xacro:chilitag_visual_sized name="chilitag29" size="${chilitag_size}">
+  <!--        <origin xyz="${chilitag_28_x} ${chilitag_28_y} ${chilitag_28_z}" rpy="0 ${-M_PI/2} 0"/>-->
+          <origin xyz="${chilitag_29_x} ${chilitag_29_y} ${chilitag_29_z}" rpy="${M_PI} ${0} ${-M_PI/2}"/>
+        </xacro:chilitag_visual_sized>
+      </xacro:if>
       <!-- Computer box-->
       <xacro:unless value="$(arg add_containment_self_filter_geom)">
@@ -262,7 +262,9 @@
     </link>
     <!-- Chilitags -->
-    <xacro:chilitag_no_geom name="chilitag29" size="${chilitag_size}" parent="${name}_link">
-      <origin xyz="${chilitag_29_x} ${chilitag_29_y} ${chilitag_29_z}" rpy="${M_PI} ${0} ${-M_PI/2}"/>
-    </xacro:chilitag_no_geom>
+    <xacro:if value="${add_chilitags}">
+      <xacro:chilitag_no_geom name="chilitag29" size="${chilitag_size}" parent="${name}_link">
+        <origin xyz="${chilitag_29_x} ${chilitag_29_y} ${chilitag_29_z}" rpy="${M_PI} ${0} ${-M_PI/2}"/>
+      </xacro:chilitag_no_geom>
+    </xacro:if>
     <!-- IMU -->
     <joint name="imu_link_joint" type="fixed">

Commit message: Update from hector_quadrotor

File: hector_models/hector_components_description/urdf/autonomy_box.urdf.xacro (robot description, xacro)
@@ -12,5 +12,5 @@
   <xacro:property name="computer_box_length" value="0.19"/>
   <xacro:property name="top_protection_bottom" value="0.4425"/>
-  <xacro:property name="insta360_mounting_height" value="0.58"/>
+  <xacro:property name="insta360_mounting_height" value="${top_protection_bottom + alu_profile_side_length + 0.12}"/>
   <xacro:property name="insta360_radius" value="0.011"/>
   <xacro:property name="insta360_collision_radius" value="0.04"/>
@@ -250,5 +250,5 @@
         </material>
       </collision>
-      <collision>
+<!--      <collision>
         <origin xyz="-0.18 0 ${computer_box_height/2+0.07}" rpy="0 0 0"/>
         <geometry>
@@ -258,5 +258,5 @@
           <color rgba="0.5 0.5 0.5 1"/>
         </material>
-      </collision>
+      </collision>-->
       </xacro:if>
     </link>
@@ -277,5 +277,5 @@
     <!-- Spinning VLP16 -->
     <xacro:spinning_sensor_mount_macro parent="${name}_link"  name="spin_lidar" scaling="0.001">
-      <origin xyz="0 0 ${0.27 + 0.0944673}" rpy="0.0 0.0 0.0"/>
+      <origin xyz="0 0 ${0.27 + 0.0944673 - 0.029}" rpy="0.0 0.0 0.0"/>
     </xacro:spinning_sensor_mount_macro>
     <!-- 360 camera -->

File: hector_models/hector_sensors_description/urdf/realsense_d435_camera.urdf.xacro (robot description, xacro)
@@ -9,8 +9,15 @@
 -->
 <robot xmlns:xacro="http://ros.org/wiki/xacro">
-    <xacro:property name="M_PI" value="3.1415926535897931" />
+  <xacro:property name="M_PI" value="3.1415926535897931" />
+  <xacro:property name="realsense_d435_width" value="0.09"/>
+  <xacro:property name="realsense_d435_height" value="0.025"/>
+  <xacro:property name="realsense_d435_depth" value="0.025"/>
+  <xacro:property name="realsense_d435_front_to_depth" value="0.0042" />
+  <xacro:property name="realsense_d435_case_offset_x" value="${realsense_d435_front_to_depth - realsense_d435_depth/2.0}"/>
+  <xacro:property name="realsense_d435_case_offset_y" value="-0.0175"/>
+  <xacro:property name="realsense_d435_case_offset_z" value="0.0"/>
     <!--
-     This macro only adds the model, it does not also add
-     the openni gazebo plugin. See the 'asus_camera' macro below for that
+     This macro only adds the model, it does not also add the openni gazebo plugin.
+     The origin is the left infrared (depth) camera, which is also the origin of the depth image
     -->
     <xacro:macro name="realsense_d435_camera_model" params="name parent *origin">
@@ -27,8 +34,7 @@
         </inertial>
         <visual>
-          <origin xyz="-0.02 -0.0325 0" rpy="0 0 0" />
+          <origin xyz="${realsense_d435_case_offset_x} ${realsense_d435_case_offset_y} ${realsense_d435_case_offset_z}" rpy="0 0 0" />
           <geometry>
-            <!--Dimensions taken from https://click.intel.com/intelr-realsensetm-depth-camera-d435.html-->
-            <box size="0.025 0.09 0.025" />
+            <box size="${realsense_d435_depth} ${realsense_d435_width} ${realsense_d435_height}" />
           </geometry>
           <material name="DarkGrey">
@@ -36,9 +42,15 @@
           </material>
         </visual>
+<!--        <visual>
+          <origin xyz="${realsense_d435_front_to_depth} ${realsense_d435_case_offset_y} 0.0" rpy="${M_PI/2} 0 ${M_PI/2}" />
+          <geometry>
+            <mesh filename="package://realsense2_camera/meshes/d435.dae" />
+          </geometry>
+        </visual>-->
         <collision>
-          <origin xyz="-0.02 -0.0325 0" rpy="0 0 0" />
+          <origin xyz="${realsense_d435_case_offset_x} ${realsense_d435_case_offset_y} ${realsense_d435_case_offset_z}" rpy="0 0 0" />
           <geometry>
             <!--Dimensions taken from https://click.intel.com/intelr-realsensetm-depth-camera-d435.html-->
-            <box size="0.025 0.09 0.025" />
+            <box size="${realsense_d435_depth} ${realsense_d435_width} ${realsense_d435_height}" />
           </geometry>
         </collision>
