Commit message: Remove misplaced issues and update hector_quadrotor

File: hector_models/hector_components_description/urdf/autonomy_box.urdf.xacro (robot description, xacro)
@@ -5,11 +5,12 @@
   <xacro:include filename="$(find hector_components_description)/urdf/vlp16_mount.urdf.xacro.xml"/>
   <xacro:include filename="$(find hector_sensors_description)/urdf/camera360.urdf.xacro"/>
+  <xacro:include filename="$(find hector_sensors_description)/urdf/realsense_t265.urdf.xacro"/>
 <!--  <xacro:arg name="add_self_filter_geom" default="0"/>-->
   <!--<xacro:property name="add_self_filter_geom" value="${arg add_self_filter_geom}"/>-->
   <xacro:property name="alu_profile_side_length" value="0.02"/>
-  <xacro:property name="computer_box_height" value="0.121"/>
+  <xacro:property name="computer_box_height" value="0.119"/>
   <xacro:property name="computer_box_width" value="0.19"/>
   <xacro:property name="computer_box_length" value="0.19"/>
-  <xacro:property name="top_protection_bottom" value="0.4425"/>
+  <xacro:property name="top_protection_bottom" value="${computer_box_height + 0.32}"/>
   <xacro:property name="insta360_mounting_height" value="${top_protection_bottom + alu_profile_side_length + 0.12}"/>
   <xacro:property name="insta360_radius" value="0.011"/>
@@ -17,4 +18,6 @@
   <xacro:property name="M_PI" value="3.14159265359"/>
   <xacro:macro name="autonomy_box_macro" params="parent *origin alu_profile_collision_size_factor name:='autonomy_box' imu_link='imu_link' add_chilitags:='true'">
+    <xacro:arg name="add_containment_self_filter_geom" default="false"/>
+    <xacro:arg name="add_manipulation_geom" default="false"/>
     <xacro:if value="${add_chilitags}">
       <xacro:include filename="$(find hector_chilitag_description)/urdf/chilitag.urdf.xacro"/>
@@ -25,5 +28,4 @@
       <xacro:property name="chilitag_29_z" value="${top_protection_bottom + alu_profile_side_length + chilitag_thickness}"/>
     </xacro:if>
-    <xacro:arg name="add_containment_self_filter_geom" default="false"/>
     <joint name="${name}_joint" type="fixed">
       <xacro:insert_block name="origin"/>
@@ -239,4 +241,16 @@
         </material>
       </collision>
+      <xacro:if value="$(arg add_manipulation_geom)">
+        <!-- Lidar protection geom -->
+        <collision>
+          <origin xyz="0 0 ${computer_box_height + 0.5*(top_protection_bottom - computer_box_height)}" rpy="0 0 0"/>
+          <geometry>
+            <cylinder length="${top_protection_bottom - computer_box_height}" radius="${computer_box_width / 2.0}"/>
+          </geometry>
+          <material name="Grey">
+            <color rgba="0.5 0.5 0.5 1"/>
+          </material>
+        </collision>
+      </xacro:if>
       </xacro:unless>
       <xacro:if value="$(arg add_containment_self_filter_geom)">
@@ -277,5 +291,5 @@
     <!-- Spinning VLP16 -->
     <xacro:spinning_sensor_mount_macro parent="${name}_link"  name="spin_lidar" scaling="0.001">
-      <origin xyz="0 0 ${0.27 + 0.0944673 - 0.029}" rpy="0.0 0.0 0.0"/>
+      <origin xyz="0 0 0.34708" rpy="0.0 0.0 0.0"/>
     </xacro:spinning_sensor_mount_macro>
     <!-- 360 camera -->
@@ -286,4 +300,22 @@
       <origin xyz="0.002862424041614364  -0.00013127655875068252 -0.03724378451297336" rpy="-3.1402707 0.0036289 -3.1175768"/> <!-- insta #3 -->
     </xacro:camera360>
+    <!-- Realsense T265 Tracking camera -->
+    <xacro:realsense_t265_tracking_camera name="tracking_camera" parent="${name}_link">
+      <origin xyz="${computer_box_width/2.0 - realsense_t265_depth/2.0} ${computer_box_width/2.0 - alu_profile_side_length - realsense_t265_width/2.0} ${top_protection_bottom - realsense_t265_height/2.0}" rpy="0 0 0"/>
+    </xacro:realsense_t265_tracking_camera>
+    <!-- +++++ Cage Realsenses +++++ -->
+    <xacro:property name="autonomy_box_realsense_x_offset" value="0.07187"/>
+    <xacro:property name="autonomy_box_realsense_y_offset" value="0.03"/>
+    <xacro:property name="autonomy_box_realsense_z_offset" value="0.00395"/>
+<!--     <xacro:property name="autonomy_box_realsense_z_offset" value="0.46895"/> -->
+    <xacro:property name="autonomy_box_realsense_pitch" value="${25*M_PI/180.0}"/>
+    <!-- Realsense D435 front -->
+    <xacro:realsense_d435_camera_with_mount_comprehensive_params name="front_rgbd_cam" parent="${name}_link" image_topic="image_rect_color" depth_points_topic="depth/color/points" min_range="0.3" max_range="9.0" update_rate="20">
+      <origin xyz="${autonomy_box_realsense_x_offset} ${-1 * autonomy_box_realsense_y_offset} ${top_protection_bottom + alu_profile_side_length + autonomy_box_realsense_z_offset}" rpy="0.0 ${autonomy_box_realsense_pitch} 0"/>
+    </xacro:realsense_d435_camera_with_mount_comprehensive_params>
+    <!-- Realsense D435 back -->
+    <xacro:realsense_d435_camera_with_mount_comprehensive_params name="back_rgbd_cam" parent="${name}_link" image_topic="image_rect_color" depth_points_topic="depth/color/points" min_range="0.3" max_range="9.0" update_rate="20">
+      <origin xyz="${-1 * autonomy_box_realsense_x_offset} ${autonomy_box_realsense_y_offset} ${top_protection_bottom + alu_profile_side_length + autonomy_box_realsense_z_offset}" rpy="0.0 ${autonomy_box_realsense_pitch} ${M_PI}"/>
+    </xacro:realsense_d435_camera_with_mount_comprehensive_params>
     <gazebo reference="${name}_link">
       <visual>

File: hector_models/hector_sensors_description/urdf/realsense_d435_camera.urdf.xacro (robot description, xacro)
@@ -13,7 +13,8 @@
   <xacro:property name="realsense_d435_height" value="0.025"/>
   <xacro:property name="realsense_d435_depth" value="0.025"/>
-  <xacro:property name="realsense_d435_front_to_depth" value="0.0042" />
+  <xacro:property name="realsense_d435_front_to_depth" value="0.0042" /> <!-- Intel_RealSense_D400_Family_Datasheet_Jan2019.pdf, page 64 -->
+  <xacro:property name="realsense_d435_mount_hole_to_front" value="0.0149" /> <!-- Measured from CAD file -->
   <xacro:property name="realsense_d435_case_offset_x" value="${realsense_d435_front_to_depth - realsense_d435_depth/2.0}"/>
-  <xacro:property name="realsense_d435_case_offset_y" value="-0.0175"/>
+  <xacro:property name="realsense_d435_case_offset_y" value="-0.0175"/> <!-- mounting hole to depth frame, Intel_RealSense_D400_Family_Datasheet_Jan2019.pdf, page 66 -->
   <xacro:property name="realsense_d435_case_offset_z" value="0.0"/>
     <!--
@@ -22,4 +23,5 @@
     -->
     <xacro:macro name="realsense_d435_camera_model" params="name parent *origin">
+      <xacro:arg name="add_raycast_self_filter_geom" default="false"/>
       <joint name="${name}_joint" type="fixed">
         <xacro:insert_block name="origin" />
@@ -55,8 +57,28 @@
           </geometry>
         </collision>
+      <xacro:if value="$(arg add_raycast_self_filter_geom)">
+        <collision>
+          <origin xyz="${realsense_d435_case_offset_x} ${realsense_d435_case_offset_y} ${realsense_d435_case_offset_z}" rpy="${M_PI*0.5} 0 0" />
+          <geometry>
+            <cylinder length="0.09" radius="0.0177"/>
+          </geometry>
+        </collision>
+      </xacro:if>
       </link>
       <gazebo reference="${name}_link">
         <material>Gazebo/Grey</material>
       </gazebo>
+    </xacro:macro>
+    <xacro:macro name="realsense_d435_camera_model_with_mount" params="name parent *origin">
+      <joint name="${name}_mount_joint" type="fixed">
+        <xacro:insert_block name="origin" />
+        <parent link="${parent}"/>
+        <child link="${name}_mount_link"/>
+      </joint>
+      <link name="${name}_mount_link">
+      </link>
+      <xacro:realsense_d435_camera_model name="${name}" parent="${name}_mount_link">
+        <origin xyz="${realsense_d435_mount_hole_to_front - realsense_d435_front_to_depth} ${-realsense_d435_case_offset_y} ${realsense_d435_height/2.0}" rpy="0 0 0"/>
+      </xacro:realsense_d435_camera_model>
     </xacro:macro>
     <xacro:macro name="realsense_d435_camera_model_no_geom" params="name parent *origin">
@@ -128,3 +150,9 @@
       <xacro:realsense_d435_camera_gazebo_plugin_macro name="${name}" parent="${parent}" image_topic="${image_topic}" depth_points_topic="${depth_points_topic}" min_range="${min_range}" max_range="${max_range}" update_rate="${update_rate}"/>
     </xacro:macro>
+    <xacro:macro name="realsense_d435_camera_with_mount_comprehensive_params" params="name parent *origin image_topic depth_points_topic min_range max_range update_rate">
+      <xacro:realsense_d435_camera_model_with_mount name="${name}" parent="${parent}">
+        <xacro:insert_block name="origin" />
+      </xacro:realsense_d435_camera_model_with_mount>
+      <xacro:realsense_d435_camera_gazebo_plugin_macro name="${name}" parent="${parent}" image_topic="${image_topic}" depth_points_topic="${depth_points_topic}" min_range="${min_range}" max_range="${max_range}" update_rate="${update_rate}"/>
+    </xacro:macro>
   </robot>

File: hector_models/hector_sensors_description/urdf/realsense_t265.urdf.xacro (robot description, xacro)
@@ -58,10 +58,16 @@
     </xacro:macro>
     <xacro:macro name="realsense_t265_tracking_camera_no_geom" params="name parent *origin">
-      <joint name="${name}_joint" type="fixed">
+      <joint name="${name}_pose_joint" type="fixed">
         <xacro:insert_block name="origin" />
         <parent link="${parent}"/>
-        <child link="${name}_link"/>
+        <child link="${name}_pose_frame"/>
       </joint>
-      <link name="${name}_link"/>
+      <link name="${name}_pose_frame"/>
+      <joint name="${name}_pose_joint2" type="fixed">
+        <origin rpy="${M_PI/2} 0 ${-M_PI/2}"/>
+        <parent link="${name}_pose_frame"/>
+        <child link="${name}_pose_frame_alt"/>
+      </joint>
+      <link name="${name}_pose_frame_alt"/>
     </xacro:macro>
   </robot>
