Commit message: Remove laser scanner and add Asus 3D sensor

File: urs_wearable/urdf/quadrotor.gazebo.xacro (robot description, xacro)
@@ -1,5 +1,5 @@
 <?xml version="1.0"?>
 <robot name="quadrotor" xmlns:xacro="http://www.ros.org/wiki/xacro">
-    <xacro:include filename="$(find urs_wearable)/urdf/quadrotor.urdf.xacro" />
-    <xacro:include filename="$(find hector_quadrotor_gazebo)/urdf/quadrotor_plugins.gazebo.xacro" />
+	<xacro:include filename="$(find urs_wearable)/urdf/quadrotor.urdf.xacro" />
+	<xacro:include filename="$(find hector_quadrotor_gazebo)/urdf/quadrotor_plugins.gazebo.xacro" />
 </robot>

File: urs_wearable/urdf/quadrotor.urdf.xacro (robot description, xacro)
@@ -1,18 +1,17 @@
 <?xml version="1.0"?>
 <robot name="quadrotor" xmlns:xacro="http://www.ros.org/wiki/xacro">
-    <xacro:property name="M_PI" value="3.1415926535897931" />
-    <!-- Included URDF Files -->
-    <xacro:include filename="$(find urs_wearable)/urdf/quadrotor_base.urdf.xacro" />
-    <!-- Instantiate quadrotor_base_macro once (has no parameters atm) -->
-    <xacro:quadrotor_base_macro />
-    <!-- Hokuyo UTM-30LX mounted upside down below the quadrotor body -->
-    <xacro:include filename="$(find hector_sensors_description)/urdf/hokuyo_utm30lx.urdf.xacro" />
-    <xacro:hokuyo_utm30lx name="laser0" parent="base_link" ros_topic="scan" update_rate="40" ray_count="1081" min_angle="-135" max_angle="135">
-      <origin xyz="0.0 0.0 -0.097" rpy="${M_PI} 0 0"/>
-    </xacro:hokuyo_utm30lx>
-    <!-- Forward facing camera -->
-    <xacro:include filename="$(find hector_sensors_description)/urdf/generic_camera.urdf.xacro" />
-    <xacro:generic_camera name="front_cam" parent="base_link" ros_topic="camera/image" cam_info_topic="camera/camera_info" update_rate="10" res_x="320" res_y="240" image_format="R8G8B8" hfov="90">
-      <origin xyz="0.05 0.0 -0.06" rpy="0 0 0"/>
-    </xacro:generic_camera>
+	<xacro:property name="M_PI" value="3.1415926535897931" />
+	<!-- Included URDF Files -->
+	<xacro:include filename="$(find hector_quadrotor_description)/urdf/quadrotor_base.urdf.xacro" />
+	<!-- Instantiate quadrotor_base_macro once (has no parameters atm) -->
+	<xacro:quadrotor_base_macro />
+	<!-- Asus Xiton Live Pro -->
+	<xacro:include filename="$(find hector_sensors_description)/urdf/asus_camera.urdf.xacro" />
+	<xacro:asus_camera name="camera" parent="base_link">
+	  <origin xyz="0.1 0.0 -0.03" rpy="0 ${M_PI/9} 0"/>
+	</xacro:asus_camera>
+	<!-- Sonar height sensor (upward) -->
+	<xacro:sonar_sensor name="sonar_upward" parent="base_link" ros_topic="sonar_upward" update_rate="10" min_range="0.03" max_range="3.0" field_of_view="${40*pi/180}" ray_count="3">
+	  <origin xyz="0.0 0.0 0.04" rpy="0 ${270*pi/180} 0"/>
+	</xacro:sonar_sensor>
 </robot>

Commit message: Replace tabs with spaces

File: urs_wearable/urdf/quadrotor.gazebo.xacro (robot description, xacro)
@@ -1,5 +1,5 @@
 <?xml version="1.0"?>
 <robot name="quadrotor" xmlns:xacro="http://www.ros.org/wiki/xacro">
-	<xacro:include filename="$(find urs_wearable)/urdf/quadrotor.urdf.xacro" />
-	<xacro:include filename="$(find hector_quadrotor_gazebo)/urdf/quadrotor_plugins.gazebo.xacro" />
+  <xacro:include filename="$(find urs_wearable)/urdf/quadrotor.urdf.xacro" />
+  <xacro:include filename="$(find hector_quadrotor_gazebo)/urdf/quadrotor_plugins.gazebo.xacro" />
 </robot>

File: urs_wearable/urdf/quadrotor.urdf.xacro (robot description, xacro)
@@ -1,17 +1,17 @@
 <?xml version="1.0"?>
 <robot name="quadrotor" xmlns:xacro="http://www.ros.org/wiki/xacro">
-	<xacro:property name="M_PI" value="3.1415926535897931" />
-	<!-- Included URDF Files -->
-	<xacro:include filename="$(find hector_quadrotor_description)/urdf/quadrotor_base.urdf.xacro" />
-	<!-- Instantiate quadrotor_base_macro once (has no parameters atm) -->
-	<xacro:quadrotor_base_macro />
-	<!-- Asus Xiton Live Pro -->
-	<xacro:include filename="$(find hector_sensors_description)/urdf/asus_camera.urdf.xacro" />
-	<xacro:asus_camera name="camera" parent="base_link">
-	  <origin xyz="0.1 0.0 -0.03" rpy="0 ${M_PI/9} 0"/>
-	</xacro:asus_camera>
-	<!-- Sonar height sensor (upward) -->
-	<xacro:sonar_sensor name="sonar_upward" parent="base_link" ros_topic="sonar_upward" update_rate="10" min_range="0.03" max_range="3.0" field_of_view="${40*pi/180}" ray_count="3">
-	  <origin xyz="0.0 0.0 0.04" rpy="0 ${270*pi/180} 0"/>
-	</xacro:sonar_sensor>
+  <xacro:property name="M_PI" value="3.1415926535897931" />
+  <!-- Included URDF Files -->
+  <xacro:include filename="$(find hector_quadrotor_description)/urdf/quadrotor_base.urdf.xacro" />
+  <!-- Instantiate quadrotor_base_macro once (has no parameters atm) -->
+  <xacro:quadrotor_base_macro />
+  <!-- Asus Xiton Live Pro -->
+  <xacro:include filename="$(find hector_sensors_description)/urdf/asus_camera.urdf.xacro" />
+  <xacro:asus_camera name="camera" parent="base_link">
+    <origin xyz="0.1 0.0 -0.03" rpy="0 ${M_PI/9} 0"/>
+  </xacro:asus_camera>
+  <!-- Sonar height sensor (upward) -->
+  <xacro:sonar_sensor name="sonar_upward" parent="base_link" ros_topic="sonar_upward" update_rate="10" min_range="0.03" max_range="3.0" field_of_view="${40*pi/180}" ray_count="3">
+    <origin xyz="0.0 0.0 0.04" rpy="0 ${270*pi/180} 0"/>
+  </xacro:sonar_sensor>
 </robot>
