Commit message: - Add collision avoidance to the controller - Integrate with FF - Small refactoring

File: urs_wearable/urdf/quadrotor.urdf.xacro (robot description, xacro)
@@ -9,5 +9,6 @@
   <xacro:include filename="$(find hector_sensors_description)/urdf/asus_camera.urdf.xacro" />
   <xacro:asus_camera name="camera" parent="base_link">
-    <origin xyz="0.1 0.0 -0.03" rpy="0 ${M_PI/9} 0"/>
+    <!-- <origin xyz="0.1 0.0 -0.03" rpy="0 ${M_PI/9} 0"/> -->
+    <origin xyz="0.1 0.0 -0.03" rpy="0 0 0"/>
   </xacro:asus_camera>
   <!-- Sonar height sensor (upward) -->
